Commit message: FIxed lidar and camera code, as well as updated lidar to have a 3D lidar. Test contains block of code for 2D lidar.

File: description/camera.xacro (robot description, xacro)
@@ -1,59 +1,52 @@
 <?xml version="1.0"?>
-<robot xmlns:xacro="http://www.ros.org/wiki/xacro">
-<joint name="camera_joint" type="fixed">
-<parent link="chassis"/>
-<child link="camera_link"/>
-<origin xyz="0.305 0 0.08" rpy="0 0 0"/>
-</joint>
-<link name="camera_link">
-<visual>
-<geometry>
-<box size="0.01 0.03 0.03"/>
-</geometry>
-<material name="red"/>
-</visual>
-<collision>
-<geometry>
-<cylinder radius="0.05" length="0.04"/>
-</geometry>
-</collision>
-<xacro:inertial_cylinder mass="0.1" length="0.04" radius="0.05">
-<origin xyz="0 0 0" rpy="0 0 0"/>
-</xacro:inertial_cylinder>
-</link>
-<joint name="camera_optical_joint" type="fixed">
-<parent link="camera_link"/>
-<child link="optical_camera_link"/>
-<origin xyz="0 0 0" rpy="$(-pi/2) 0 $(-pi/2)"/>
-</joint>
-<gazebo reference="camera_link">
-<material>Gazebo/Red</material>
-<!-- <sensor name="laser" type="ray">
-<pose>0 0 0 0 0 0</pose>
-<visualize>true</visualize>
-<update_rate>10</update_rate>
-<ray>
-<scan>
-<horizontal>
-<samples>360</samples>
-<resolution>1</resolution>
-<min_angle>-3.14</min_angle>
-<max_angle>3.14</max_angle>
-</horizontal>
-</scan>
-<range>
-<min>0.3</min>
-<max>12</max>
-<resolution>0.01</resolution>
-</range>
-</ray>
-<plugin name="laser_controller" filename="libgazebo_ros_ray_sensor.so">
-<ros>
-<argument>~/out:=scan</argument>
-</ros>
-<output_type>sensor_msgs/LaserScan</output_type>
-<frame_name>laser_frame</frame_name>
-</plugin>
-</sensor> -->
-</gazebo>
+<robot xmlns:xacro="http://www.ros.org/wiki/xacro" >
+    <joint name="camera_joint" type="fixed">
+        <parent link="chassis"/>
+        <child link="camera_link"/>
+        <origin xyz="0.276 0 0.181" rpy="0 0.18 0"/>
+    </joint>
+    <link name="camera_link">
+        <visual>
+            <geometry>
+                <box size="0.010 0.03 0.03"/>
+            </geometry>
+            <material name="black"/>
+        </visual>
+        <visual>
+            <origin xyz="0 0 -0.05"/>
+            <geometry>
+                <cylinder radius="0.002" length="0.1"/>
+            </geometry>
+            <material name="black"/>
+        </visual>
+    </link>
+    <joint name="camera_optical_joint" type="fixed">
+        <parent link="camera_link"/>
+        <child link="camera_link_optical"/>
+        <origin xyz="0 0 0" rpy="${-pi/2} 0 ${-pi/2}"/>
+    </joint>
+    <link name="camera_link_optical"></link>
+    <gazebo reference="camera_link">
+        <material>Gazebo/Black</material>
+        <sensor name="camera" type="camera">
+            <pose> 0 0 0 0 0 0 </pose>
+            <visualize>true</visualize>
+            <update_rate>120</update_rate>
+            <camera>
+                <horizontal_fov>1.089</horizontal_fov>
+                <image>
+                    <format>R8G8B8</format>
+                    <width>1280</width>
+                    <height>720</height>
+                </image>
+                <clip>
+                    <near>0.05</near>
+                    <far>8.0</far>
+                </clip>
+            </camera>
+            <plugin name="camera_controller" filename="libgazebo_ros_camera.so">
+                <frame_name>camera_link_optical</frame_name>
+            </plugin>
+        </sensor>
+    </gazebo>
 </robot>

File: description/lidar.xacro (robot description, xacro)
@@ -23,32 +23,43 @@
     </link>
     <gazebo reference="laser_frame">
-        <material>Gazebo/Red</material>
-            <sensor name="laser" type="ray">
-                <pose>0 0 0 0 0 0</pose>
-                <visualize>true</visualize>
-                <update_rate>10</update_rate>
-                <ray>
+    <material>Gazebo/Red</material>
+        <sensor name="lidar3d" type="gpu_lidar">
+            <pose>0 0 0 0 0 0</pose>
+            <visualize>true</visualize>
+            <update_rate>120</update_rate>
+            <ray>
                 <scan>
-                <horizontal>
-                <samples>360</samples>
-                <resolution>1</resolution>
-                <min_angle>-3.14</min_angle>
-                <max_angle>3.14</max_angle>
-                </horizontal>
+                    <horizontal>
+                        <samples>360</samples>
+                        <resolution>1</resolution>
+                        <min_angle>-3.14</min_angle>
+                        <max_angle>3.14</max_angle>
+                    </horizontal>
+                    <vertical>
+                        <samples>48</samples>
+                        <resolution>1</resolution>
+                        <min_angle>-0.3</min_angle>
+                        <max_angle>0.3</max_angle>
+                    </vertical>
                 </scan>
-<range>
-<min>0.3</min>
-<max>12</max>
-<resolution>0.01</resolution>
-</range>
-</ray>
-<plugin name="laser_controller" filename="libgazebo_ros_ray_sensor.so">
-<ros>
-<argument>~/out:=scan</argument>
-</ros>
-<output_type>sensor_msgs/LaserScan</output_type>
-<frame_name>laser_frame</frame_name>
-</plugin>
-</sensor>
-</gazebo>
+                <range>
+                    <min>0.3</min>
+                    <max>12</max>
+                    <resolution>0.01</resolution>
+                </range>
+                <noise>
+                    <type>gaussian</type>
+                    <mean>0.0</mean>
+                    <stddev>0.01</stddev>
+                </noise>
+            </ray>
+            <plugin name="lidar3d_plugin" filename="libgazebo_ros_ray_sensor.so">
+                <ros>
+                    <argument>~/out:=lidar_points</argument>
+                </ros>
+                <topicName>lidar_points</topicName>
+                <frame_name>laser_frame</frame_name>
+            </plugin>
+        </sensor>
+    </gazebo>
 </robot>

File: description/robot.urdf.xacro (robot description, xacro)
@@ -4,3 +4,5 @@
     <xacro:include filename="gazebo_control.xacro" />
     <xacro:include filename="lidar.xacro" />
+    <xacro:include filename="camera.xacro" />
+    <!-- <xacro:include filename="depth_camera.xacro" /> -->
 </robot>
