Commit message: Fixed LiDAR issue not working in Rviz and successfully able to SLAM

File: description/lidar.xacro (robot description, xacro)
@@ -24,5 +24,5 @@
     <gazebo reference="laser_frame">
     <material>Gazebo/Red</material>
-        <sensor name="lidar3d" type="gpu_lidar">
+        <sensor name="laser" type="ray">
             <pose>0 0 0 0 0 0</pose>
             <visualize>true</visualize>
@@ -36,10 +36,4 @@
                         <max_angle>3.14</max_angle>
                     </horizontal>
-                    <vertical>
-                        <samples>48</samples>
-                        <resolution>1</resolution>
-                        <min_angle>-0.3</min_angle>
-                        <max_angle>0.3</max_angle>
-                    </vertical>
                 </scan>
                 <range>
@@ -48,15 +42,11 @@
                     <resolution>0.01</resolution>
                 </range>
-                <noise>
-                    <type>gaussian</type>
-                    <mean>0.0</mean>
-                    <stddev>0.01</stddev>
-                </noise>
             </ray>
-            <plugin name="lidar3d_plugin" filename="libgazebo_ros_ray_sensor.so">
+            <plugin name="laser_controller" filename="libgazebo_ros_ray_sensor.so">
                 <ros>
-                    <argument>~/out:=lidar_points</argument>
+                    <namespace>/</namespace>
+                    <remapping>~/out:=scan</remapping>
                 </ros>
-                <topicName>lidar_points</topicName>
+                <output_type>sensor_msgs/LaserScan</output_type>
                 <frame_name>laser_frame</frame_name>
             </plugin>

File: description/robot.urdf.xacro (robot description, xacro)
@@ -4,5 +4,5 @@
     <xacro:include filename="gazebo_control.xacro" />
     <xacro:include filename="lidar.xacro" />
-    <xacro:include filename="camera.xacro" />
-    <!-- <xacro:include filename="depth_camera.xacro" /> -->
+    <!-- <xacro:include filename="camera.xacro" /> -->
+    <xacro:include filename="depth_camera.xacro" />
 </robot>

File: description/robot_core.xacro (robot description, xacro)
@@ -19,4 +19,12 @@
     <!-- BASE LINK -->
     <link name="base_link">
+    </link>
+    <!-- BASE FOOTPRINT LINK -->
+    <joint name="base_footprint_joint" type="fixed">
+        <parent link="base_link"/>
+        <child link="base_footprint"/>
+        <origin xyz="0 0 0" rpy="0 0 0"/>
+    </joint>
+    <link name="base_footprint">
     </link>
     <!-- CHASSIS LINK -->
